Commit message: Add Jazzy modifications

File: rb1_ros2_description/urdf/bases/rb1_base_v3.urdf.xacro (robot description, xacro)
@@ -8,10 +8,4 @@
   <xacro:if value="${publish_bf}">
     <link name="${prefix}base_footprint">
-      <!--visual>
-          <origin xyz="0 0 0" rpy="0 0 0" />
-          <geometry>
-             <box size="0.001 0.001 0.001" />
-          </geometry>
-      </visual-->
     </link>
     <joint name="${prefix}base_footprint_joint" type="fixed">

File: rb1_ros2_description/urdf/common.gazebo.xacro (robot description, xacro)
@@ -6,5 +6,5 @@
 	<xacro:macro name="gazebo_colors" params="prefix">
 		<gazebo reference="$(arg prefix)base_footprint">
-			<material>Gazebo/Green</material>
+			<material>Gazebo/Black</material>
 		</gazebo>
 		<gazebo reference="$(arg prefix)base_link">

File: rb1_ros2_description/urdf/elevator/elevator.gazebo.xacro (robot description, xacro)
@@ -10,31 +10,5 @@
 			<material>Gazebo/Grey</material>
 			<turnGravityOff>false</turnGravityOff>
-			<!--kp>500000.0</kp>
-			<kd>10.0</kd>
-			<mu1>10</mu1>
-			<mu2>10</mu2>
-			<fdir1>1 0 0</fdir1-->
-			<!--minDepth>0.001</minDepth-->
-			<!--material>Gazebo/Black</material-->
-			<!--mu1 value="10"/>
-			<mu2 value="5"/>
-			<kp value="500000.0" />
-			<kd value="10.0" />
-			<fdir1 value="1 0 0"/>
-			<material>Gazebo/Yellow</material>
-			<turnGravityOff>false</turnGravityOff-->
 		</gazebo>
-		<!--gazebo reference="${name}_wheel_link">
-			<kp>500000.0</kp>
-			<kd>10.0</kd>
-			<mu1>10</mu1>
-			<mu2>10</mu2>
-			<fdir1>1 0 0</fdir1>
-			<maxVel>1.0</maxVel>
-			<minDepth>0.003</minDepth>
-			<material>Gazebo/Yellow</material>
-			<turnGravityOff>false</turnGravityOff>
-			<implicitSpringDamper>1</implicitSpringDamper>
-		</gazebo-->
 	</xacro:macro>
 </robot>

File: rb1_ros2_description/urdf/wheels/omni_wheel.gazebo.xacro (robot description, xacro)
@@ -8,4 +8,5 @@
 			<kd value="1.0" />
 			<fdir1 value="1 0 0"/>
+            <material>Gazebo/Yellow</material>
 			<turnGravityOff>false</turnGravityOff>
 		</gazebo>

File: rb1_ros2_description/urdf/wheels/omni_wheel.urdf.xacro (robot description, xacro)
@@ -14,5 +14,4 @@
   <xacro:macro name="omni_wheel" params="prefix parent *origin hq">
 <!--WHEEL TIRE -->
-    <!-- joint name="joint_${name}_wheel" type="continuous" -->
     <joint name="${prefix}wheel_joint" type="fixed">
       <parent link="${parent}"/>
@@ -65,19 +64,7 @@
 		<kd value="1.0" />
 		<fdir1 value="1 0 0"/>
-		<material>Gazebo/Black</material>
+		<!--<material>Gazebo/Black</material>-->
 		<turnGravityOff>false</turnGravityOff>
     </gazebo>
-    <!--gazebo reference="${name}_wheel">
-		<kp>500000.0</kp>
-		<kd>10.0</kd>
-		<mu1>10</mu1>
-		<mu2>10</mu2>
-		<fdir1>1 0 0</fdir1>
-		<maxVel>1.0</maxVel>
-		<minDepth>0.003</minDepth>
-		<material>Gazebo/Black</material>
-		<turnGravityOff>false</turnGravityOff>
-		<implicitSpringDamper>1</implicitSpringDamper>
-    </gazebo-->
   </xacro:macro>
 </robot>

File: rb1_ros2_description/urdf/wheels/rubber_wheel.gazebo.xacro (robot description, xacro)
@@ -10,31 +10,5 @@
 			<material>Gazebo/Yellow</material>
 			<turnGravityOff>false</turnGravityOff>
-			<!--kp>500000.0</kp>
-			<kd>10.0</kd>
-			<mu1>10</mu1>
-			<mu2>10</mu2>
-			<fdir1>1 0 0</fdir1-->
-			<!--minDepth>0.001</minDepth-->
-			<!--material>Gazebo/Black</material-->
-			<!--mu1 value="10"/>
-			<mu2 value="5"/>
-			<kp value="500000.0" />
-			<kd value="10.0" />
-			<fdir1 value="1 0 0"/>
-			<material>Gazebo/Yellow</material>
-			<turnGravityOff>false</turnGravityOff-->
 		</gazebo>
-		<!--gazebo reference="${name}_wheel_link">
-			<kp>500000.0</kp>
-			<kd>10.0</kd>
-			<mu1>10</mu1>
-			<mu2>10</mu2>
-			<fdir1>1 0 0</fdir1>
-			<maxVel>1.0</maxVel>
-			<minDepth>0.003</minDepth>
-			<material>Gazebo/Yellow</material>
-			<turnGravityOff>false</turnGravityOff>
-			<implicitSpringDamper>1</implicitSpringDamper>
-		</gazebo-->
 	</xacro:macro>
 </robot>

File: rb1_ros2_description/xacro/rb1_ros2_base.urdf.xacro (robot description, xacro)
@@ -12,6 +12,6 @@
 	<xacro:include filename="$(find rb1_ros2_description)/urdf/wheels/rubber_wheel.urdf.xacro" />
 	<xacro:include filename="$(find rb1_ros2_description)/urdf/wheels/omni_wheel.urdf.xacro" />
-	<!-- Import all available sensors -->
-	<xacro:include filename="$(find rb1_ros2_description)/urdf/all_sensors.urdf.xacro" />
+	<!-- Import all available sensors -->¡
+    <xacro:include filename="$(find robotnik_sensors)/urdf/all_sensors.urdf.xacro" />
 	<!-- Import Gazebo Stuff -->
 	<xacro:include filename="$(find rb1_ros2_description)/urdf/common.gazebo.xacro" />
@@ -75,13 +75,7 @@
 	</xacro:elevator_platform>
 	<!-- SENSORS -->
-	<xacro:sensor_hokuyo_ust20lx prefix="$(arg prefix)front_laser" parent="$(arg prefix)base_link" prefix_topic="front_laser" gpu="$(arg gpu)">
+	<xacro:sensor_hokuyo_ust20lx frame_prefix="$(arg prefix)front_laser_" parent="$(arg prefix)base_link" topic_prefix="front_laser" gpu="$(arg gpu)">
 		<origin xyz="0.210 0.0 0.21" rpy="0 3.1416 3.1416"/>
 	</xacro:sensor_hokuyo_ust20lx>
-	<xacro:sensor_imu_hector prefix="$(arg prefix)imu" parent="$(arg prefix)base_link">
-		<origin xyz="0.002 0.053 0.1485" rpy="0 0 0"/>
-	</xacro:sensor_imu_hector>
-	<xacro:sensor_orbbec_astra prefix="$(arg prefix)front_rgbd_camera" parent="$(arg prefix)base_link" prefix_topic="front_rgbd_camera">
-		<origin xyz="0.234 0.0 0.092" rpy="0 0 0"/>
-	</xacro:sensor_orbbec_astra>
 	<!-- Gazebo ros2 control plugins -->
 	<!-- <xacro:ros2_control/> -->
