Commit message: WIP: wire RB-1 ros2_control and Gazebo plugin

File: rb1_ros2_description/xacro/rb1_ros2_base.urdf.xacro (robot description, xacro)
@@ -80,3 +80,23 @@
 	<!-- Gazebo ros2 control plugins -->
 	<!-- <xacro:ros2_control/> -->
+    <!-- CP15-C014: Learner control block (default prefix robot_). -->
+    <ros2_control name="diff_drive" type="system">
+        <hardware>
+            <plugin>gz_ros2_control/GazeboSimSystem</plugin>
+        </hardware>
+        <joint name="robot_left_wheel_joint">
+            <command_interface name="velocity"/>
+            <state_interface name="velocity"/>
+        </joint>
+        <joint name="robot_right_wheel_joint">
+            <command_interface name="velocity"/>
+            <state_interface name="velocity"/>
+        </joint>
+    </ros2_control>
+    <!-- CP15-C015: Learner Gazebo plugin configuration. -->
+    <gazebo>
+        <plugin filename="gz_ros2_control-system" name="gz_ros2_control::GazeboSimROS2ControlPlugin">
+            <parameters>$(find rb1_ros2_description)/config/rb1_controller.yaml</parameters>
+        </plugin>
+    </gazebo>
 </robot>

Commit message: Configure RB-1 elevator position controller

File: rb1_ros2_description/xacro/rb1_ros2_base.urdf.xacro (robot description, xacro)
@@ -95,4 +95,8 @@
             <state_interface name="position"/>
         </joint>
+        <joint name="robot_elevator_platform_joint">
+            <command_interface name="position"/>
+            <state_interface name="position"/>
+        </joint>
     </ros2_control>
     <!-- CP15-C015: Learner Gazebo plugin configuration. -->
